File: 4MB/gvpsimm.kicad_sch (KiCad schematic)
At the start: 18 parts, among them J1 SIMM64_EDGE, U1 HM514400_alt, U2 HM514400_alt, U3 HM514400_alt, U4 HM514400_alt, U5 HM514400_alt, U6 HM514400_alt, U7 HM514400_alt, U8 HM514400_alt

Commit message: Modify license
Other:
- note added: "This project is licensed under the CERN Open Hardware License Version 2 - Permissive."
- note removed: "This work is licensed under the Creative Commons Attribution-ShareAlike 4.0 International License. To view a copy of this license, visit http://creativecommons.org/licenses/by-sa/4.0/ or send a letter to Creative Commons, PO Box 1866, Mountain View, CA 94042, USA"
